Commit message: June 24th Morning

File: my_mobile/install/my_robot_description/share/my_robot_description/urdf/robot_core.xacro (robot description, xacro)
@@ -33,4 +33,5 @@
         <child link="left_wheel"/>
         <origin xyz="0 ${wheel_separation/2} 0" rpy="0 0 0"/>
+        <axis xyz="0 1 0"/>
     </joint>
     <link name="left_wheel">
