Commit message: June 26th

File: my_mobile/src/my_robot_description/urdf/robot.urdf.xacro (robot description, xacro)
@@ -3,5 +3,6 @@
     <xacro:include filename="robot_core.xacro"/>
     <xacro:include filename="robot_gazebo.xacro"/>
-    <!-- <xacro:include filename="gazebo_control.xacro"/> -->
     <xacro:include filename="ros2_control.xacro" />
+    <xacro:include filename="lidar.xacro" />
+    <xacro:include filename="camera.xacro"/>
 </robot>

File: my_mobile/src/my_robot_description/urdf/robot_core.xacro (robot description, xacro)
@@ -1,5 +1,4 @@
 <?xml version="1.0"?>
-<robot name="my_mobile"
-    xmlns:xacro="http://www.ros.org/wiki/xacro">
+<robot name="my_mobile" xmlns:xacro="http://www.ros.org/wiki/xacro">
     <xacro:property name="wheel_separation" value="0.180"/>
     <xacro:property name="wheel_diameter" value="0.068"/>
@@ -10,6 +9,6 @@
         <origin xyz="0 0 ${wheel_diameter/2}" rpy="0 0 0"/>
     </joint>
-    <link name="base_link">
-        <visual>
+	<link name="base_link">
+		<visual>
             <origin xyz="0 0 0" rpy="0 0 0"/>
             <geometry>
@@ -28,5 +27,5 @@
             <inertia ixx="0.01" ixy="0" ixz="0" iyy="0.01" iyz="0" izz="0.01"/>
         </inertial>
-    </link>
+	</link>
     <joint name="left_wheel_joint" type="continuous">
         <parent link="base_link"/>
